Commit message: Updated joint transforms to match CAD

File: q_pup_config/urdf/quadruped.urdf (robot description, URDF)
Before this commit: robot quadruped, 21 links, 20 joints
Joints:
- joint lf_debug_joint: origin xyz=0.3149 0.2384 0 rpy=0 0 0 -> xyz=0.3174 0.2384 0 rpy=0 0 0
- joint lf_foot_joint: origin xyz=0.0 0.0 -0.35 rpy=0 0 0 -> xyz=0.0 0.0 -0.353 rpy=0 0 0
- joint lf_hip_joint: origin xyz=0.3149 0.2384 0.0 rpy=0 0 0 -> xyz=0.3174 0.2384 0.0 rpy=0 0 0
- joint lf_upper_leg_joint: origin xyz=0.0906 0.0815 -0.0 rpy=0 0 0 -> xyz=0.0881 0.0825 -0.0 rpy=0 0 0
- joint lh_debug_joint: origin xyz=-0.3149 0.2384 0 rpy=0 0 0 -> xyz=-0.3174 0.2384 0 rpy=0 0 0
- joint lh_foot_joint: origin xyz=0.0 0.0 -0.35 rpy=0 0 0 -> xyz=0.0 0.0 -0.353 rpy=0 0 0
- joint lh_hip_joint: origin xyz=-0.3149 0.2384 0.0 rpy=0 0 0 -> xyz=-0.3174 0.2384 0.0 rpy=0 0 0
- joint lh_upper_leg_joint: origin xyz=-0.0906 0.0815 -0.0 rpy=0 0 0 -> xyz=-0.0881 0.0825 -0.0 rpy=0 0 0
- joint rf_debug_joint: origin xyz=0.3149 -0.2384 0 rpy=0 0 0 -> xyz=0.3174 -0.2384 0 rpy=0 0 0
- joint rf_foot_joint: origin xyz=0.0 0.0 -0.35 rpy=0 0 0 -> xyz=0.0 0.0 -0.353 rpy=0 0 0
- joint rf_hip_joint: origin xyz=0.3149 -0.2384 0.0 rpy=0 0 0 -> xyz=0.3174 -0.2384 0.0 rpy=0 0 0
- joint rf_upper_leg_joint: origin xyz=0.0906 -0.0815 -0.0 rpy=0 0 0 -> xyz=0.0881 -0.0825 -0.0 rpy=0 0 0
- joint rh_debug_joint: origin xyz=-0.3149 -0.2384 0 rpy=0 0 0 -> xyz=-0.3174 -0.2384 0 rpy=0 0 0
- joint rh_foot_joint: origin xyz=0.0 0.0 -0.35 rpy=0 0 0 -> xyz=0.0 0.0 -0.353 rpy=0 0 0
- joint rh_hip_joint: origin xyz=-0.3149 -0.2384 0.0 rpy=0 0 0 -> xyz=-0.3174 -0.2384 0.0 rpy=0 0 0
- joint rh_upper_leg_joint: origin xyz=-0.0906 -0.0815 -0.0 rpy=0 0 0 -> xyz=-0.0881 -0.0825 -0.0 rpy=0 0 0
