Commit message: RE FAC TOR

File: qpup_config/urdf/quadruped.urdf (robot description, URDF)
Before this commit: robot quadruped, 21 links, 20 joints
Joints:
- removed joint lf_hip_joint
- removed joint lf_lower_leg_joint
- removed joint lf_upper_leg_joint
- removed joint lh_hip_joint
- removed joint lh_lower_leg_joint
- removed joint lh_upper_leg_joint
- removed joint rf_hip_joint
- removed joint rf_lower_leg_joint
- removed joint rf_upper_leg_joint
- removed joint rh_hip_joint
- removed joint rh_lower_leg_joint
- removed joint rh_upper_leg_joint
- added joint FLH: type revolute, parent lf_hip_link, child lf_upper_leg_link, origin xyz=0.0881 0.0825 -0.0 rpy=0 0 0, axis 0 1 0, limit lower=-3.14159265359 upper=3.14159265359 effort=25 velocity=1.5
- added joint FLK: type revolute, parent lf_upper_leg_link, child lf_lower_leg_link, origin xyz=0.0 0.0 -0.4 rpy=0 0 0, axis 0 1 0, limit lower=-3.14159265359 upper=3.14159265359 effort=25 velocity=1.5
- added joint FLS: type revolute, parent base_link, child lf_hip_link, origin xyz=0.3174 0.2384 0.0 rpy=0 0 0, axis 1 0 0, limit lower=-3.14159265359 upper=3.14159265359 effort=25 velocity=1.5
- added joint FRH: type revolute, parent rf_hip_link, child rf_upper_leg_link, origin xyz=0.0881 -0.0825 -0.0 rpy=0 0 0, axis 0 1 0, limit lower=-3.14159265359 upper=3.14159265359 effort=25 velocity=1.5
- added joint FRK: type revolute, parent rf_upper_leg_link, child rf_lower_leg_link, origin xyz=0.0 0.0 -0.4 rpy=0 0 0, axis 0 1 0, limit lower=-3.14159265359 upper=3.14159265359 effort=25 velocity=1.5
- added joint FRS: type revolute, parent base_link, child rf_hip_link, origin xyz=0.3174 -0.2384 0.0 rpy=0 0 0, axis 1 0 0, limit lower=-3.14159265359 upper=3.14159265359 effort=25 velocity=1.5
- added joint RLH: type revolute, parent lh_hip_link, child lh_upper_leg_link, origin xyz=-0.0881 0.0825 -0.0 rpy=0 0 0, axis 0 1 0, limit lower=-3.14159265359 upper=3.14159265359 effort=25 velocity=1.5
- added joint RLK: type revolute, parent lh_upper_leg_link, child lh_lower_leg_link, origin xyz=0.0 0.0 -0.4 rpy=0 0 0, axis 0 1 0, limit lower=-3.14159265359 upper=3.14159265359 effort=25 velocity=1.5
- added joint RLS: type revolute, parent base_link, child lh_hip_link, origin xyz=-0.3174 0.2384 0.0 rpy=0 0 0, axis 1 0 0, limit lower=-3.14159265359 upper=3.14159265359 effort=25 velocity=1.5
- added joint RRH: type revolute, parent rh_hip_link, child rh_upper_leg_link, origin xyz=-0.0881 -0.0825 -0.0 rpy=0 0 0, axis 0 1 0, limit lower=-3.14159265359 upper=3.14159265359 effort=25 velocity=1.5
- added joint RRK: type revolute, parent rh_upper_leg_link, child rh_lower_leg_link, origin xyz=0.0 0.0 -0.4 rpy=0 0 0, axis 0 1 0, limit lower=-3.14159265359 upper=3.14159265359 effort=25 velocity=1.5
- added joint RRS: type revolute, parent base_link, child rh_hip_link, origin xyz=-0.3174 -0.2384 0.0 rpy=0 0 0, axis 1 0 0, limit lower=-3.14159265359 upper=3.14159265359 effort=25 velocity=1.5
